Commit message: feat:增加moveit示例

File: ros2/smrcore_description/urdf/smri3.ros2_control.xacro (robot description, xacro)
@@ -1,11 +1,25 @@
 <?xml version="1.0"?>
 <robot xmlns:xacro="http://www.ros.org/wiki/xacro">
-  <xacro:macro name="smri3_ros2_control" params="robot_ip">
+  <xacro:macro name="smri3_ros2_control" params="robot_ip hardware_backend:=real log_passthrough_commands:=false">
     <ros2_control name="smrcore_hardware" type="system">
-      <hardware>
-        <plugin>smrcore_hardware/SMRcoreSystemInterface</plugin>
-        <param name="robot_ip">${robot_ip}</param>
-      </hardware>
-      <joint name="joint1">
+      <xacro:if value="${hardware_backend == 'real'}">
+        <hardware>
+          <plugin>smrcore_hardware/SMRcoreSystemInterface</plugin>
+          <param name="robot_ip">${robot_ip}</param>
+          <param name="log_passthrough_commands">${log_passthrough_commands}</param>
+        </hardware>
+      </xacro:if>
+      <xacro:if value="${hardware_backend == 'mock'}">
+        <hardware>
+          <plugin>mock_components/GenericSystem</plugin>
+          <param name="calculate_dynamics">false</param>
+        </hardware>
+      </xacro:if>
+      <xacro:if value="${hardware_backend == 'gazebo'}">
+        <hardware>
+          <plugin>gazebo_ros2_control/GazeboSystem</plugin>
+        </hardware>
+      </xacro:if>
+      <joint name="base_joint">
         <command_interface name="position"/>
         <command_interface name="velocity"/>
@@ -14,5 +28,5 @@
         <state_interface name="effort"/>
       </joint>
-      <joint name="joint2">
+      <joint name="shoulder_joint">
         <command_interface name="position"/>
         <command_interface name="velocity"/>
@@ -21,5 +35,5 @@
         <state_interface name="effort"/>
       </joint>
-      <joint name="joint3">
+      <joint name="elbow_joint">
         <command_interface name="position"/>
         <command_interface name="velocity"/>
@@ -28,5 +42,5 @@
         <state_interface name="effort"/>
       </joint>
-      <joint name="joint4">
+      <joint name="wrist1_joint">
         <command_interface name="position"/>
         <command_interface name="velocity"/>
@@ -35,5 +49,5 @@
         <state_interface name="effort"/>
       </joint>
-      <joint name="joint5">
+      <joint name="wrist2_joint">
         <command_interface name="position"/>
         <command_interface name="velocity"/>
@@ -42,5 +56,5 @@
         <state_interface name="effort"/>
       </joint>
-      <joint name="joint6">
+      <joint name="wrist3_joint">
         <command_interface name="position"/>
         <command_interface name="velocity"/>

File: ros2/smrcore_description/urdf/smri3.urdf.xacro (robot description, xacro)
@@ -2,4 +2,6 @@
 <robot name="smri3" xmlns:xacro="http://www.ros.org/wiki/xacro">
   <xacro:arg name="robot_ip" default=""/>
+  <xacro:arg name="hardware_backend" default="real"/>
+  <xacro:arg name="log_passthrough_commands" default="false"/>
   <xacro:include filename="$(find smrcore_description)/urdf/materials.xacro"/>
   <xacro:include filename="$(find smrcore_description)/urdf/smrcore_macro.xacro"/>
@@ -29,5 +31,5 @@
   <xacro:smrcore_link name="link6" radius="0.035" length="0.12" color="smrcore_light"/>
   <link name="tool0"/>
-  <joint name="joint1" type="revolute">
+  <joint name="base_joint" type="revolute">
     <parent link="base_link"/>
     <child link="link1"/>
@@ -36,5 +38,5 @@
     <limit lower="-6.283185307" upper="6.283185307" effort="200" velocity="3.14"/>
   </joint>
-  <joint name="joint2" type="revolute">
+  <joint name="shoulder_joint" type="revolute">
     <parent link="link1"/>
     <child link="link2"/>
@@ -43,5 +45,5 @@
     <limit lower="-6.283185307" upper="6.283185307" effort="200" velocity="3.14"/>
   </joint>
-  <joint name="joint3" type="revolute">
+  <joint name="elbow_joint" type="revolute">
     <parent link="link2"/>
     <child link="link3"/>
@@ -50,5 +52,5 @@
     <limit lower="-6.283185307" upper="6.283185307" effort="200" velocity="3.14"/>
   </joint>
-  <joint name="joint4" type="revolute">
+  <joint name="wrist1_joint" type="revolute">
     <parent link="link3"/>
     <child link="link4"/>
@@ -57,5 +59,5 @@
     <limit lower="-6.283185307" upper="6.283185307" effort="120" velocity="3.14"/>
   </joint>
-  <joint name="joint5" type="revolute">
+  <joint name="wrist2_joint" type="revolute">
     <parent link="link4"/>
     <child link="link5"/>
@@ -64,5 +66,5 @@
     <limit lower="-6.283185307" upper="6.283185307" effort="120" velocity="3.14"/>
   </joint>
-  <joint name="joint6" type="revolute">
+  <joint name="wrist3_joint" type="revolute">
     <parent link="link5"/>
     <child link="link6"/>
@@ -76,4 +78,4 @@
     <origin xyz="0 0 0.12" rpy="0 0 0"/>
   </joint>
-  <xacro:smri3_ros2_control robot_ip="$(arg robot_ip)"/>
+  <xacro:smri3_ros2_control robot_ip="$(arg robot_ip)" hardware_backend="$(arg hardware_backend)" log_passthrough_commands="$(arg log_passthrough_commands)"/>
 </robot>

Commit message: feat: 测试中文路径下的gazebo问题

File: ros2/smrcore_description/urdf/smri3.ros2_control.xacro (robot description, xacro)
@@ -23,6 +23,12 @@
       <joint name="base_joint">
         <command_interface name="position"/>
-        <command_interface name="velocity"/>
-        <state_interface name="position"/>
+        <xacro:unless value="${hardware_backend == 'gazebo'}">
+          <command_interface name="velocity"/>
+        </xacro:unless>
+        <state_interface name="position">
+          <xacro:if value="${hardware_backend == 'gazebo'}">
+            <param name="initial_value">0.0</param>
+          </xacro:if>
+        </state_interface>
         <state_interface name="velocity"/>
         <state_interface name="effort"/>
@@ -30,6 +36,12 @@
       <joint name="shoulder_joint">
         <command_interface name="position"/>
-        <command_interface name="velocity"/>
-        <state_interface name="position"/>
+        <xacro:unless value="${hardware_backend == 'gazebo'}">
+          <command_interface name="velocity"/>
+        </xacro:unless>
+        <state_interface name="position">
+          <xacro:if value="${hardware_backend == 'gazebo'}">
+            <param name="initial_value">0.0</param>
+          </xacro:if>
+        </state_interface>
         <state_interface name="velocity"/>
         <state_interface name="effort"/>
@@ -37,6 +49,12 @@
       <joint name="elbow_joint">
         <command_interface name="position"/>
-        <command_interface name="velocity"/>
-        <state_interface name="position"/>
+        <xacro:unless value="${hardware_backend == 'gazebo'}">
+          <command_interface name="velocity"/>
+        </xacro:unless>
+        <state_interface name="position">
+          <xacro:if value="${hardware_backend == 'gazebo'}">
+            <param name="initial_value">0.0</param>
+          </xacro:if>
+        </state_interface>
         <state_interface name="velocity"/>
         <state_interface name="effort"/>
@@ -44,6 +62,12 @@
       <joint name="wrist1_joint">
         <command_interface name="position"/>
-        <command_interface name="velocity"/>
-        <state_interface name="position"/>
+        <xacro:unless value="${hardware_backend == 'gazebo'}">
+          <command_interface name="velocity"/>
+        </xacro:unless>
+        <state_interface name="position">
+          <xacro:if value="${hardware_backend == 'gazebo'}">
+            <param name="initial_value">0.0</param>
+          </xacro:if>
+        </state_interface>
         <state_interface name="velocity"/>
         <state_interface name="effort"/>
@@ -51,6 +75,12 @@
       <joint name="wrist2_joint">
         <command_interface name="position"/>
-        <command_interface name="velocity"/>
-        <state_interface name="position"/>
+        <xacro:unless value="${hardware_backend == 'gazebo'}">
+          <command_interface name="velocity"/>
+        </xacro:unless>
+        <state_interface name="position">
+          <xacro:if value="${hardware_backend == 'gazebo'}">
+            <param name="initial_value">0.0</param>
+          </xacro:if>
+        </state_interface>
         <state_interface name="velocity"/>
         <state_interface name="effort"/>
@@ -58,6 +88,12 @@
       <joint name="wrist3_joint">
         <command_interface name="position"/>
-        <command_interface name="velocity"/>
-        <state_interface name="position"/>
+        <xacro:unless value="${hardware_backend == 'gazebo'}">
+          <command_interface name="velocity"/>
+        </xacro:unless>
+        <state_interface name="position">
+          <xacro:if value="${hardware_backend == 'gazebo'}">
+            <param name="initial_value">0.0</param>
+          </xacro:if>
+        </state_interface>
         <state_interface name="velocity"/>
         <state_interface name="effort"/>

File: ros2/smrcore_description/urdf/smri3_real.urdf.xacro (robot description, xacro)
@@ -7,4 +7,5 @@
   <xacro:arg name="hardware_backend" default="real"/>
   <xacro:arg name="log_passthrough_commands" default="false"/>
+  <xacro:arg name="gazebo_controllers_file" default="$(find smrcore_hardware)/config/smri3_gazebo_controllers.yaml"/>
   <xacro:property name="hardware_backend_value" value="$(arg hardware_backend)"/>
   <xacro:include filename="$(find smrcore_description)/urdf/smri3.ros2_control.xacro"/>
@@ -417,12 +418,12 @@
         rpy="0 0 0" />
       <mass
-        value="0" />
-      <inertia
-        ixx="0"
+        value="0.001" />
+      <inertia
+        ixx="1e-06"
         ixy="0"
         ixz="0"
-        iyy="0"
+        iyy="1e-06"
         iyz="0"
-        izz="0" />
+        izz="1e-06" />
     </inertial>
     <visual>
@@ -463,9 +464,26 @@
       xyz="0 0 0" />
   </joint>
+  <xacro:if value="${hardware_backend_value == 'gazebo'}">
+    <!-- Keep Gazebo's URDF root inertial-free without changing the default
+         exported tree used by RViz, MoveIt, and the real hardware backend. -->
+    <link name="world"/>
+    <joint name="world_to_base_link" type="fixed">
+      <parent link="world"/>
+      <child link="base_link"/>
+      <origin xyz="0 0 0" rpy="0 0 0"/>
+    </joint>
+  </xacro:if>
   <xacro:smri3_ros2_control robot_ip="$(arg robot_ip)" hardware_backend="$(arg hardware_backend)" log_passthrough_commands="$(arg log_passthrough_commands)"/>
   <xacro:if value="${hardware_backend_value == 'gazebo'}">
+    <gazebo reference="base_link">
+      <!-- The exported base collision mesh slightly intersects the ground and
+           the arm has no external fixture in URDF. Keep the base kinematic in
+           Gazebo so position-control tests do not drift or chatter. -->
+      <gravity>false</gravity>
+      <kinematic>true</kinematic>
+    </gazebo>
     <gazebo>
       <plugin filename="libgazebo_ros2_control.so" name="gazebo_ros2_control">
-        <parameters>$(find smrcore_hardware)/config/smri3_controllers.yaml</parameters>
+        <parameters>$(arg gazebo_controllers_file)</parameters>
       </plugin>
     </gazebo>
